File: pcb/Drawdio_v10.sch (EAGLE design)
At the start: 14 parts, among them IC1 TLC551, Q1 BC327

Commit message: cleaned up schematics and layout
Other:
- note added: "Based on the work of Jay Silver (www.drawdio.com)"
- note added: "and Ladyada (www.adafruit.com)"
- note removed: "Based on the work of Jay Silver (www.drawdio.com) and Ladyada (www.adafruit.com)"
Changed lines of the file:
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@@
 <setting verticaltext="up"/>
 </settings>
-<grid distance="0.1" unitdist="inch" unit="inch" style="lines" multiple="1" display="no" altdistance="0.01" altunitdist="inch" altunit="inch"/>
+<grid distance="0.05" unitdist="inch" unit="inch" style="lines" multiple="1" display="yes" altdistance="0.025" altunitdist="inch" altunit="inch"/>
 <layers>
 <layer number="1" name="Top" color="4" fill="1" visible="no" active="no"/>
@@
 <part name="R3" library="rcl-ez" deviceset="R-US_" device="0207/10" value="10M"/>
 <part name="U$1" library="drawdio" deviceset="AAA" device=""/>
-<part name="FRAME1" library="frames" deviceset="A4L-LOC" device=""/>
+<part name="FRAME1" library="we-symbol" deviceset="FRAME-A4L" device=""/>
 </parts>
 <sheets>
@@
 <wire x1="96.52" y1="114.3" x2="101.6" y2="114.3" width="0.1524" layer="95"/>
 <circle x="99.06" y="119.38" radius="2.54" width="0.1524" layer="95"/>
-<text x="161.29" y="34.29" size="1.27" layer="95">Released under the Creative Commons Attribution Share-Alike License</text>
-<text x="161.29" y="31.75" size="1.27" layer="95">http://creativecommons.org/licenses/by-sa/4.0/</text>
-<text x="161.29" y="27.94" size="1.27" layer="95">Designed by Stephan Watterott (Watterott electronic)</text>
-<text x="161.29" y="25.4" size="1.27" layer="95">Based on the work of Jay Silver (www.drawdio.com) and Ladyada (www.adafruit.com)</text>
+<text x="162.56" y="21.59" size="1.27" layer="95">Released under the Creative Commons Attribution Share-Alike License</text>
+<text x="162.56" y="19.05" size="1.27" layer="95">http://creativecommons.org/licenses/by-sa/4.0/</text>
+<text x="162.56" y="15.24" size="1.27" layer="95">Designed by Stephan Watterott (Watterott electronic)</text>
+<text x="162.56" y="12.7" size="1.27" layer="95">Based on the work of Jay Silver (www.drawdio.com)</text>
 <text x="34.29" y="146.05" size="2.54" layer="95">Drawdio is an electronic pencil that makes music while you draw. It is a simple musical synthesizer
 that uses the conductive properties of pencil graphite to create different sounds.
 The result is a fun toy that lets you draw musical instruments on any piece of paper.
 The original design/idea is from Jay Silver.</text>
+<text x="162.56" y="10.16" size="1.27" layer="95">and Ladyada (www.adafruit.com)</text>
 </plain>
 <instances>
